Commit message: ing

File: hw3/ur_description/urdf/ur5_original.urdf (robot description, URDF)
Before this commit: robot universal_robot, 8 links, 7 joints
Joints:
- joint shoulder_pan_joint: type fixed -> revolute
- joint wrist_1_joint: type fixed -> revolute
- joint wrist_2_joint: type fixed -> revolute
- joint wrist_3_joint: type fixed -> revolute
