Commit message: sim

File: hw3/ur_description/urdf/ur5.urdf (robot description, URDF)
Before this commit: robot universal_robot, 8 links, 7 joints
Joints:
- joint shoulder_pan_joint: type revolute -> fixed
- joint wrist_1_joint: type revolute -> fixed
- joint wrist_2_joint: type revolute -> fixed
- joint wrist_3_joint: type revolute -> fixed

Commit message: hw3

File: hw3/ur_description/urdf/ur5.urdf (robot description, URDF)
Before this commit: robot universal_robot, 8 links, 7 joints
Links:
- link base_link: geometry collision mesh filename=../meshes/ur5/collision/base.dae; visual mesh filename=../meshes/ur5/visual/base.dae
- link forearm_link: geometry collision mesh filename=../meshes/ur5/collision/forearm.dae; visual mesh filename=../meshes/ur5/visual/forearm.dae
- link shoulder_link: geometry collision mesh filename=../meshes/ur5/collision/shoulder.dae; visual mesh filename=../meshes/ur5/visual/shoulder.dae
- link upper_arm_link: geometry collision mesh filename=../meshes/ur5/collision/upperarm.dae; visual mesh filename=../meshes/ur5/visual/upperarm.dae
- link wrist_1_link: geometry collision mesh filename=../meshes/ur5/collision/wrist1.dae; visual mesh filename=../meshes/ur5/visual/wrist1.dae
- link wrist_2_link: geometry collision mesh filename=../meshes/ur5/collision/wrist2.dae; visual mesh filename=../meshes/ur5/visual/wrist2.dae
- link wrist_3_link: geometry collision mesh filename=../meshes/ur5/collision/wrist3.dae; visual mesh filename=../meshes/ur5/visual/wrist3.dae

Commit message: ing

File: hw3/ur_description/urdf/ur5.urdf (robot description, URDF)
Before this commit: robot universal_robot, 8 links, 7 joints
Links:
- removed link ee_link
- removed link wrist_1_link
- removed link wrist_2_link
- removed link wrist_3_link
Joints:
- removed joint ee_fixed_joint
- removed joint wrist_1_joint
- removed joint wrist_2_joint
- removed joint wrist_3_joint

Commit message: ing

File: hw3/ur_description/urdf/ur5.urdf (robot description, URDF)
Before this commit: robot universal_robot, 4 links, 3 joints
Links:
- link shoulder_link: mass 3.7 -> 0.0

Commit message: HW3 complete

File: hw3/ur_description/urdf/ur5.urdf (robot description, URDF)
Before this commit: robot universal_robot, 8 links, 7 joints
Links:
- removed link ee_link
- link base_link: mass 4.0 -> 0.0
- link shoulder_link: mass 3.7 -> 0.0
- link wrist_1_link: mass 1.219 -> 0.0
- link wrist_2_link: mass 1.219 -> 0.0
- link wrist_3_link: mass 0.1879 -> 0.0
Joints:
- removed joint ee_fixed_joint
