Commit message: rsdRobot

File: hw3/ur_description/urdf/ur3.urdf (robot description, URDF)
Before this commit: robot UR3, 7 links, 6 joints
Links:
- link base_link: geometry collision mesh filename=../meshes/ur3/collision/base.stl; visual mesh filename=../meshes/ur3/visual/base.stl
- link forearm_link: geometry collision mesh filename=../meshes/ur3/collision/forearm.stl; visual mesh filename=../meshes/ur3/visual/forearm.stl
- link shoulder_link: geometry collision mesh filename=../meshes/ur3/collision/shoulder.stl; visual mesh filename=../meshes/ur3/visual/shoulder.stl
- link upper_arm_link: geometry collision mesh filename=../meshes/ur3/collision/upperarm.stl; visual mesh filename=../meshes/ur3/visual/upperarm.stl
- link wrist_1_link: geometry collision mesh filename=../meshes/ur3/collision/wrist1.stl; visual mesh filename=../meshes/ur3/visual/wrist1.stl
- link wrist_2_link: geometry collision mesh filename=../meshes/ur3/collision/wrist2.stl; visual mesh filename=../meshes/ur3/visual/wrist2.stl
- link wrist_3_link: geometry collision mesh filename=../meshes/ur3/collision/wrist3.stl; visual mesh filename=../meshes/ur3/visual/wrist3.stl
