Commit message: urdf changed

File: rsdrobot_description/urdf/rsdRobot.xacro (robot description, xacro)
@@ -190,7 +190,8 @@
     <link name="ee_link">
         <visual>
-            <origin xyz="0 0 -0.075"/>
+            <origin xyz="0 0 -0.0632"/>
             <geometry>
                 <mesh filename="package://rsdrobot_description/meshes/ee.dae" scale="0.001 0.001 0.001"/>
+                <!-- <sphere radius="0.01"/> -->
             </geometry>
             <material name="LightGrey"/>

Commit message: 221201

File: rsdrobot_description/urdf/rsdRobot.xacro (robot description, xacro)
@@ -69,5 +69,5 @@
         <parent link="joint1_link"/>
         <child link="joint2_link"/>
-        <origin xyz="0.070 0.000 0.075" rpy="1.570796 0.0 0.0"/>
+        <origin xyz="0.070 0.000 0.0753" rpy="1.570796 0.0 0.0"/>
         <axis xyz="0 0 1"/>
         <limit lower="-3.141592" upper="3.141592" effort="100.0" velocity="100.0"/>
@@ -169,5 +169,5 @@
             <origin xyz="0 0 0"/>
             <geometry>
-                <sphere radius="0.01"/>
+                <sphere radius="0.001"/>
             </geometry>
             <material name="LightGrey"/>
